Commit message: Working Controller

File: urdf/arm.urdf (robot description, URDF)
Before this commit: robot robotic_arm, 5 links, 4 joints
Joints:
- joint base_joint: axis (none) -> 0.0 0.0 1.0; origin (none) -> xyz=0.0 0.0 0.0 rpy=0.0 0.0 0.0

Commit message: Switched to Trajectory Controller

File: urdf/arm.urdf (robot description, URDF)
Before this commit: robot robotic_arm, 5 links, 4 joints
Links:
- link base_link: geometry collision cylinder length=0.05 radius=0.1; visual cylinder length=0.05 radius=0.1
